Commit message: Add the workflow, and the hardware the workflow needs
The task module is the only one that knows what order things happen in, and
everything it calls is a capability that does not know it is part of a
sequence. Writing it surfaced what the arm was still missing.

The kind of glass is now decided from the side-on measurement rather than from
the overhead view. A kind here is a shape, and the measured profile is a
description of that shape, so a handful of tests read it off and the project
needs no trained classifier. It is also more honest: from above, a stem is
invisible and a tall glass looks like a short one, so a glass classified from
overhead can be handed a rule its shape cannot support.

For the same reason the overhead detection no longer reports a height. It
reports the footprint width, measured by putting both edges of the blob on the
table rather than by scaling pixels, and the side view supplies everything else.

The gripper grew what handling glass requires:

  - silicone pads, which conform to a curved wall instead of touching it at one
    point, and which are where the 6 degree slope tolerance comes from;
  - an effort command interface and a second controller, because holding a
    glass is a force job and a position controller would keep driving towards
    a number the glass is in the way of;
  - a force sensor at the wrist, which is the only way to learn what a glass
    weighs, since wall thickness is not visible from outside.

Turning a glass over is a rotation about the grip, not a move to a pose, so
the arm gained rotate_tool and does it about the one point on the glass that
is not moving relative to the fingers. Which way round to hold a glass is
settled before the fingers close, by checking the turn can be made from there:
the last wrist joint stops short of a full turn, and finding that out with the
glass already held leaves nothing to do but put it back.

141 tests pass.

Co-Authored-By: Claude Opus 5 <noreply@anthropic.com>
Claude-Session: https://claude.ai/code/session_014pENzTX8Fwof2SgoRfagAu

File: v5-pick-glasses/src/work_cell/work_cell/arm/arm.urdf.xacro (robot description, xacro)
@@ -48,4 +48,28 @@
     </joint>
   </xacro:macro>
+  <!--
+    The fingers offer two ways of being commanded, and the task uses both.
+    Position is for opening the gripper and for closing it to a width the
+    measurement has worked out. Effort is for holding: once the pads are on the
+    glass, what matters is how hard they press, and a position controller
+    cannot express that. It would keep driving towards a number the glass is in
+    the way of.
+    Only one controller may hold a joint at a time, so the two are swapped
+    between during the run. arm/motion.py does the swapping.
+  -->
+  <xacro:macro name="finger_joint" params="name initial:=0.0">
+    <joint name="${name}">
+      <command_interface name="position"/>
+      <command_interface name="effort">
+        <param name="min">-25.0</param>
+        <param name="max">25.0</param>
+      </command_interface>
+      <state_interface name="position">
+        <param name="initial_value">${initial}</param>
+      </state_interface>
+      <state_interface name="velocity"/>
+      <state_interface name="effort"/>
+    </joint>
+  </xacro:macro>
   <ros2_control name="work_cell_system" type="system">
     <hardware>
@@ -59,6 +83,18 @@
     <xacro:position_joint name="wrist_2_joint" initial="-1.5708"/>
     <xacro:position_joint name="wrist_3_joint" initial="0.0"/>
-    <xacro:position_joint name="left_finger_joint" initial="0.04"/>
-    <xacro:position_joint name="right_finger_joint" initial="0.04"/>
+    <xacro:finger_joint name="left_finger_joint" initial="0.0475"/>
+    <xacro:finger_joint name="right_finger_joint" initial="0.0475"/>
+    <!-- The wrist force sensor, as ros2_control sees it. The broadcaster reads
+         these and publishes a WrenchStamped; the sensor itself is declared on
+         the gripper mount in arm/gripper.urdf.xacro. -->
+    <sensor name="wrist_force">
+      <state_interface name="force.x"/>
+      <state_interface name="force.y"/>
+      <state_interface name="force.z"/>
+      <state_interface name="torque.x"/>
+      <state_interface name="torque.y"/>
+      <state_interface name="torque.z"/>
+      <param name="frame_id">gripper_body</param>
+    </sensor>
   </ros2_control>
   <gazebo>

File: v5-pick-glasses/src/work_cell/work_cell/arm/gripper.urdf.xacro (robot description, xacro)
@@ -2,18 +2,25 @@
 <robot xmlns:xacro="http://wiki.ros.org/xacro">
   <!--
-    A two-finger parallel gripper.
-    Both fingers are driven independently rather than one mimicking the other,
-    because a mimic joint has to be handled by the simulated hardware as well
-    as by the model, and two joints commanded to the same number needs nothing
-    special from anybody. Closed, the two fingers meet and act as a single
-    blunt tip, which is what touches the face of a cuboid.
+    A two-finger parallel gripper with soft pads, and a force sensor at the
+    wrist.
+    Three things about this gripper exist because it handles glass.
+    The pads are silicone rather than bare metal. A rigid pad touches a curved
+    glass wall at one point, and all of the grip force goes through that point.
+    A soft pad spreads over a small patch instead, which both holds better and
+    is what makes a slightly sloping wall safe to grip: the pad conforms to the
+    slope rather than sliding off it. The 6 degree figure in
+    glasses/profile.py comes from how much slope a 12 mm pad can take up.
+    The fingers are driven by effort as well as by position. Position alone
+    cannot hold a glass: the controller would keep driving towards a number the
+    glass is in the way of, and a thin-walled glass loses. Squeezing to a
+    commanded force is how much of the squeeze is decided, and
+    glasses/force.py decides how much.
+    A force sensor sits between the flange and the gripper. It is how the arm
+    finds out what a glass really weighs, which no camera can tell it, and how
+    it knows the rack has taken the weight before the fingers open.
     Along the tool's z axis:
       0.000  tool0, the flange
       0.050  the fingers start
       0.170  the fingertips
-    The fingers are long on purpose. To touch the side of a tall box the arm
-    comes in from above at an angle, and short fingers would bring the body of
-    the gripper down onto the top of the box before the fingertip reached the
-    face.
   -->
   <xacro:macro name="parallel_gripper" params="prefix parent">
@@ -21,8 +28,13 @@
     <xacro:property name="body_length" value="0.05"/>
     <xacro:property name="finger_length" value="0.12"/>
-    <xacro:property name="finger_thickness" value="0.012"/>
+    <xacro:property name="finger_thickness" value="0.010"/>
     <xacro:property name="finger_width" value="0.03"/>
-    <!-- Half the fingers' thickness, so travel 0 has them just touching. -->
-    <xacro:property name="finger_home" value="${finger_thickness / 2}"/>
+    <!-- The silicone pad on the inside face of each finger. Its height is what
+         decides how much upright wall a grip needs, which is PAD_HEIGHT in
+         arm/dimensions.py. -->
+    <xacro:property name="pad_thickness" value="0.004"/>
+    <xacro:property name="pad_height" value="0.014"/>
+    <!-- Half of finger plus pad, so travel 0 has the two pads just touching. -->
+    <xacro:property name="finger_home" value="${(finger_thickness + 2 * pad_thickness) / 2}"/>
     <link name="${prefix}gripper_body">
       <visual>
@@ -41,4 +53,7 @@
       </inertial>
     </link>
+    <!-- The mount is where the force sensor reads. It has to be a real joint
+         for Gazebo to put a sensor on it, which is why the gripper is not
+         simply welded to the flange. -->
     <joint name="${prefix}gripper_mount" type="fixed">
       <parent link="${parent}"/>
@@ -46,4 +61,17 @@
       <origin xyz="0 0 0"/>
     </joint>
+    <gazebo reference="${prefix}gripper_mount">
+      <sensor name="wrist_force" type="force_torque">
+        <always_on>true</always_on>
+        <update_rate>100</update_rate>
+        <force_torque>
+          <!-- Reported in the frame of the link below the joint, which is the
+               gripper. That is the frame the arm reasons in: "how hard is the
+               thing I am holding pulling along my own z axis". -->
+          <frame>child</frame>
+          <measure_direction>child_to_parent</measure_direction>
+        </force_torque>
+      </sensor>
+    </gazebo>
     <xacro:macro name="finger" params="side reflect">
       <link name="${prefix}${side}_finger">
@@ -68,42 +96,68 @@
         <origin xyz="0 ${reflect * finger_home} ${body_length}"/>
         <axis xyz="0 ${reflect} 0"/>
-        <!-- 25 N is the grip. It is far more than the few newtons needed to
-             hold a wooden block against gravity, and far less than a finger
-             driven at full strength into a box it cannot squash, which sends
-             the box shooting out sideways. -->
-        <limit lower="0.0" upper="0.04" effort="25.0" velocity="0.1"/>
+        <!-- 25 N is what the finger can push with at most. The grip actually
+             used is commanded run by run and is usually a tenth of this: see
+             glasses/force.py, where it is worked out from the weight of the
+             glass and capped by what its walls can take. -->
+        <limit lower="0.0" upper="0.0475" effort="25.0" velocity="0.1"/>
+      </joint>
+      <!-- The pad. A separate link so that it can have silicone's contact
+           properties while the finger behind it stays stiff. -->
+      <link name="${prefix}${side}_pad">
+        <visual>
+          <origin xyz="0 0 0"/>
+          <geometry><box size="${finger_width} ${pad_thickness} ${pad_height}"/></geometry>
+          <material name="pad_black"><color rgba="0.1 0.1 0.12 1"/></material>
+        </visual>
+        <collision>
+          <origin xyz="0 0 0"/>
+          <geometry><box size="${finger_width} ${pad_thickness} ${pad_height}"/></geometry>
+        </collision>
+        <inertial>
+          <mass value="0.005"/>
+          <inertia ixx="1.0e-7" ixy="0" ixz="0" iyy="1.0e-7" iyz="0" izz="1.0e-7"/>
+        </inertial>
+      </link>
+      <!-- At the fingertip end, on the inside face. -->
+      <joint name="${prefix}${side}_pad_mount" type="fixed">
+        <parent link="${prefix}${side}_finger"/>
+        <child link="${prefix}${side}_pad"/>
+        <origin xyz="0 ${-reflect * (finger_thickness + pad_thickness) / 2}
+                     ${finger_length - pad_height / 2}"/>
       </joint>
     </xacro:macro>
     <xacro:finger side="left" reflect="1"/>
     <xacro:finger side="right" reflect="-1"/>
-    <!-- Grip needs friction, and a cuboid squeezed between two frictionless
-         plates just squirts out. -->
-    <xacro:macro name="finger_surface" params="link">
+    <!-- Silicone on glass. High friction, and soft: kp is two orders of
+         magnitude below the rigid finger, which is what lets the pad flatten
+         against a curved wall instead of touching it at one point. -->
+    <xacro:macro name="pad_surface" params="link">
       <gazebo reference="${link}">
-        <mu1>1.6</mu1>
-        <mu2>1.6</mu2>
-        <kp>1e6</kp>
-        <kd>100.0</kd>
+        <mu1>1.9</mu1>
+        <mu2>1.9</mu2>
+        <kp>1e4</kp>
+        <kd>50.0</kd>
+        <minDepth>0.0005</minDepth>
       </gazebo>
     </xacro:macro>
-    <xacro:finger_surface link="${prefix}left_finger"/>
-    <xacro:finger_surface link="${prefix}right_finger"/>
-    <!-- Contact sensors on the fingers. They are what turns "the arm went to
-         where it calculated the face centre is" into "the arm felt the face".
-         Both fingers carry one, because which of the two lands on a face first
-         depends on how the box happens to be sitting. -->
-    <xacro:macro name="finger_contact" params="side">
-      <gazebo reference="${prefix}${side}_finger">
-        <sensor name="${side}_fingertip_contact" type="contact">
+    <xacro:pad_surface link="${prefix}left_pad"/>
+    <xacro:pad_surface link="${prefix}right_pad"/>
+    <!-- Contact sensors on the pads. They are what turns "the arm went to
+         where it calculated the grip height is" into "the pads are on the
+         glass", and they are also what stops the descent into a rack slot,
+         since the rim touching down is a contact and nothing else is. -->
+    <xacro:macro name="pad_contact" params="side">
+      <gazebo reference="${prefix}${side}_pad">
+        <sensor name="${side}_pad_contact" type="contact">
           <always_on>true</always_on>
           <update_rate>60</update_rate>
           <contact>
-            <collision>${prefix}${side}_finger_collision</collision>
+            <collision>${prefix}${side}_pad_collision</collision>
           </contact>
         </sensor>
       </gazebo>
     </xacro:macro>
-    <xacro:finger_contact side="left"/>
-    <xacro:finger_contact side="right"/>
+    <xacro:pad_contact side="left"/>
+    <xacro:pad_contact side="right"/>
   </xacro:macro>
 </robot>
