Commit message: The cell's hardware becomes three real products
The gripper, the wrist force sensor and the wrist camera were invented: boxes
drawn in this repo with plausible numbers. They are now a Robotiq 2F-85, a
Robotiq FT 300-S and an Intel RealSense D405, and the simulator loads the
descriptions Robotiq and Intel publish rather than anything drawn here.

Six things the real hardware decided, rather than this project choosing:

- The gripper has **one** driven joint. A 2F-85 is told a knuckle angle, not a
  finger width, so arm/robotiq_2f85.py translates between them. Everything
  else about the linkage follows from the offsets Robotiq publish, including
  the 85 mm stroke, which is now worked out rather than written down.
- **The pads swing forward as they close**, by up to 13.7 mm, because the
  fingers turn on a linkage instead of sliding. Where a glass is gripped
  therefore depends on how far shut the gripper is, so GRASP_DEPTH became
  grasp_depth(opening) and the tool is placed for the gap the fingers will
  finish at.
- **The widest glass it can hold is 80 mm, not the 85 mm it opens to.** Past
  that, a glass held at the middle of the pads reaches back and touches the
  gripper's body. spec.py had been claiming 95 mm, which no gripper in this
  cell ever did.
- **It cannot squeeze below 20 N.** The sums here ask for single newtons, so
  every glass is held several times harder than it needs. The force caps had
  to be rewritten against that floor, because against the old guesses of 6,
  12 and 20 N the gripper's own minimum broke every thin and normal glass's
  rating and the arm would have refused nearly every glass on the table.
  force.py now reports how much harder it squeezed than it meant to.
- **The UR5e's own force sensor cannot weigh a glass**, at +/-4.0 N accuracy
  against a glass weighing about 2 N, which is why an FT 300-S is bolted on
  instead of using the free one in the flange.
- **The camera could not focus on the finger view** where it was mounted: a
  D405 is blind inside 70 mm and the lens sat 37 to 66 mm from the glass wall.
  Moved to the back of the gripper body, every width the gripper can hold is
  in range.

Two consequences in the surrounding code. The survey footprint was worked out
from the tool's height while the camera now hangs 69 mm further along the
tool, which claimed nearly a third more table than the camera sees; it uses
the camera's height now. And the SRDF disables every pair among the tool's
links, because a 2F-85 is a closed linkage whose parts touch by design.

Problem 3's bench still models the old jaw, and says so in a comment: changing
it alters the physics of every push, so all six solutions would need running
again and the four trained ones training again first.

249 tests pass, lint clean, and the expanded URDF agrees with every number in
dimensions.py. Three test failures remain and all three already failed before
this change.

Co-Authored-By: Claude Opus 5 (1M context) <noreply@anthropic.com>

File: v5-pick-glasses/src/work_cell/work_cell/arm/arm.urdf.xacro (robot description, xacro)
@@ -2,9 +2,17 @@
 <robot xmlns:xacro="http://wiki.ros.org/xacro" name="work_cell">
   <!--
-    The whole robot: a UR5e standing on the table, a two-finger gripper on its
-    flange, and an RGB-D camera beside the gripper.
-    Universal Robots publish the arm itself, so ur_description supplies the
-    links, the joint limits and the calibrated link lengths for the UR5e. What
-    is added here is the tooling and the wiring to ros2_control.
+    The whole robot: a UR5e standing on the table, a Robotiq FT 300-S force
+    sensor and a Robotiq 2F-85 gripper on its flange, and an Intel RealSense
+    D405 depth camera beside the gripper.
+    Every part of it is a real product whose maker publishes its own robot
+    description, and this file's job is only to stack them and wire them to
+    ros2_control. `ur_description` supplies the UR5e's links, joint limits and
+    calibrated link lengths; `robotiq_description` supplies the gripper and
+    the coupling that bolts it to a UR flange; `realsense2_description`
+    supplies the camera. Nothing about their shapes is written here.
+    See arm/gripper.urdf.xacro for why this particular gripper and this
+    particular sensor, and arm/robotiq_2f85.py for the one thing that follows
+    from using a real gripper: it is driven by a single knuckle angle rather
+    than by a finger width.
   -->
   <xacro:arg name="ur_type" default="ur5e"/>
@@ -32,5 +40,8 @@
   </xacro:ur_robot>
   <xacro:parallel_gripper prefix="" parent="tool0"/>
-  <xacro:wrist_camera prefix="" parent="gripper_body"/>
+  <!-- On the gripper's own body, which is the link Robotiq's description calls
+       robotiq_85_base_link, so the camera rides with the gripper rather than
+       with the sensor under it. -->
+  <xacro:wrist_camera prefix="" parent="robotiq_85_base_link"/>
   <!--
     ros2_control describes the joints a controller is allowed to touch and who
@@ -49,5 +60,5 @@
   </xacro:macro>
   <!--
-    The fingers offer two ways of being commanded, and the task uses both.
+    The gripper offers two ways of being commanded, and the task uses both.
     Position is for opening the gripper and for closing it to a width the
     measurement has worked out. Effort is for holding: once the pads are on the
@@ -57,4 +68,13 @@
     Only one controller may hold a joint at a time, so the two are swapped
     between during the run. arm/motion.py does the swapping.
+    There is only **one** joint to command, which is the difference the real
+    gripper makes here. The 2F-85 has a single motor on a single knuckle, and
+    both fingers follow it through a linkage, which Robotiq's description
+    expresses as mimic joints. So this is a one-joint gripper that happens to
+    have two fingers, and the width the task thinks in is a number
+    arm/robotiq_2f85.py works out from the angle.
+    The effort limits are the ones Robotiq's description declares for that
+    joint, in newton metres at the knuckle rather than newtons at the
+    fingertip. arm/robotiq_2f85.py converts between them.
   -->
   <xacro:macro name="finger_joint" params="name initial:=0.0">
@@ -62,6 +82,6 @@
       <command_interface name="position"/>
       <command_interface name="effort">
-        <param name="min">-25.0</param>
-        <param name="max">25.0</param>
+        <param name="min">-50.0</param>
+        <param name="max">50.0</param>
       </command_interface>
       <state_interface name="position">
@@ -83,9 +103,11 @@
     <xacro:position_joint name="wrist_2_joint" initial="-1.5708"/>
     <xacro:position_joint name="wrist_3_joint" initial="0.0"/>
-    <xacro:finger_joint name="left_finger_joint" initial="0.0475"/>
-    <xacro:finger_joint name="right_finger_joint" initial="0.0475"/>
-    <!-- The wrist force sensor, as ros2_control sees it. The broadcaster reads
-         these and publishes a WrenchStamped; the sensor itself is declared on
-         the gripper mount in arm/gripper.urdf.xacro. -->
+    <!-- Wide open, which is zero on this joint and grows as it shuts. -->
+    <xacro:finger_joint name="robotiq_85_left_knuckle_joint" initial="0.0"/>
+    <!-- The FT 300-S, as ros2_control sees it. The broadcaster reads these and
+         publishes a WrenchStamped. The frame is the sensor's own link, because
+         that is where the real sensor reads: it sits on the flange and senses
+         everything bolted beyond it, which is the coupling, the gripper, the
+         camera, and whatever the fingers are holding. -->
     <sensor name="wrist_force">
       <state_interface name="force.x"/>
@@ -95,5 +117,5 @@
       <state_interface name="torque.y"/>
       <state_interface name="torque.z"/>
-      <param name="frame_id">gripper_body</param>
+      <param name="frame_id">force_sensor_link</param>
     </sensor>
   </ros2_control>

File: v5-pick-glasses/src/work_cell/work_cell/arm/camera/wrist_camera.urdf.xacro (robot description, xacro)
@@ -2,38 +2,55 @@
 <robot xmlns:xacro="http://wiki.ros.org/xacro">
   <!--
-    An RGB-D camera bolted beside the gripper, looking the same way the fingers
-    point. Because it rides on the wrist, pointing the tool at something is the
-    same as pointing the camera at it, and the arm can walk the camera around a
+    An Intel RealSense D405 depth camera bolted beside the gripper, looking the
+    same way the fingers point.
+    The shape, the mass and the frames are Intel's own: `realsense2_description`
+    ships the model, so this file includes it and adds only the mount and the
+    Gazebo sensor that renders through it.
+    The D405 is the short-range camera of the RealSense family, and that is why
+    it is the one here. Its working range is about 70 mm to 500 mm, which is
+    uncomfortably close for a mobile robot and exactly right for a camera that
+    rides on a wrist and is stood 300 mm off a glass to measure it. The other
+    common choice, the D435, starts at about 300 mm, so the closest look this
+    task takes would be at the very edge of what it can do.
+    Because it rides on the wrist, pointing the tool at something is the same
+    as pointing the camera at it, and the arm can walk the camera around a
     glass to see whether it has a handle, which one side-on view cannot show.
-    Two frames, as ROS expects for a camera:
-      wrist_camera_link           x forward, the frame Gazebo renders from
-      wrist_camera_optical_frame  z forward, x right, y down, the frame image
-                                  pixels are projected in
+    Two things about the real camera matter to the code that reads it.
+    **Its depth and colour pictures come from the same place.** Intel's own
+    description puts the colour sensor at no offset from the depth sensor on
+    this model, unlike the D435, so one optical frame serves for both and
+    glasses/perception.py can project a colour pixel and a depth pixel with the
+    same arithmetic.
+    **It sees much more than the camera this project used to assume.** The D405
+    covers about 87 degrees across, where the invented camera covered 60. That
+    changes how much table one picture holds and therefore how many places the
+    arm has to stand to survey it. Nothing in the code needed changing for it,
+    because the measurements read the focal length out of the camera's own
+    `camera_info` message rather than assuming one.
   -->
+  <xacro:include filename="$(find realsense2_description)/urdf/_d405.urdf.xacro"/>
   <xacro:macro name="wrist_camera" params="prefix parent">
-    <link name="${prefix}wrist_camera_link">
-      <visual>
-        <geometry><box size="0.025 0.05 0.02"/></geometry>
-        <material name="camera_black"><color rgba="0.1 0.1 0.1 1"/></material>
-      </visual>
-      <inertial>
-        <mass value="0.05"/>
-        <inertia ixx="1e-5" ixy="0" ixz="0" iyy="1e-5" iyz="0" izz="1e-5"/>
-      </inertial>
-    </link>
-    <!-- Out to the side of the gripper body so the fingers stay out of shot,
-         and turned a quarter turn so the camera's own x axis lies along the
-         tool's z axis. -->
-    <joint name="${prefix}wrist_camera_mount" type="fixed">
-      <parent link="${parent}"/>
-      <child link="${prefix}wrist_camera_link"/>
-      <origin xyz="0.085 0 0.015" rpy="0 ${-pi/2} 0"/>
-    </joint>
-    <link name="${prefix}wrist_camera_optical_frame"/>
-    <joint name="${prefix}wrist_camera_optical_joint" type="fixed">
-      <parent link="${prefix}wrist_camera_link"/>
-      <child link="${prefix}wrist_camera_optical_frame"/>
-      <origin xyz="0 0 0" rpy="${-pi/2} 0 ${-pi/2}"/>
-    </joint>
+    <!-- Across the fingers rather than along them, and at the back of the
+         gripper's body rather than level with its middle. Across, because the
+         fingers swing in the tool's x direction and reach about 74 mm out
+         either way when the gripper is open, so a camera mounted that way
+         would sit inside their swing; across them the widest thing is the
+         gripper's own 75 mm body. At the back, because this camera cannot
+         focus closer than about 70 mm and the closest look it takes is down
+         the fingers at a glass they are already round. The reasoning, and the
+         distances it comes out at, are in arm/dimensions.py beside
+         CAMERA_MOUNT. Turned a quarter turn so the camera looks along the
+         tool's z axis, which is the direction the fingers point. -->
+    <!-- The optical frames are optional in Intel's description and are off by
+         default, because on real hardware the camera driver publishes better
+         ones from the calibration stored in the device. In simulation there is
+         no device to read, so the nominal frames are what there is, and the
+         measurements need one: glasses/perception.py projects pixels in it. -->
+    <xacro:sensor_d405
+      parent="${parent}"
+      name="${prefix}wrist_camera"
+      use_nominal_extrinsics="true">
+      <origin xyz="0 0.050 0.010" rpy="0 ${-pi/2} ${-pi/2}"/>
+    </xacro:sensor_d405>
     <gazebo reference="${prefix}wrist_camera_link">
       <sensor name="wrist_camera" type="rgbd_camera">
@@ -42,19 +59,35 @@
         <topic>wrist_camera</topic>
         <camera>
-          <horizontal_fov>1.047</horizontal_fov>
-          <!-- 320x240 keeps the colour and depth frames small enough to cross
-               the ROS bridge comfortably, and from the height the arm looks
-               from one pixel still covers under 1.5 mm of table, which is finer
-               than the millimetre the measurements are reported to. -->
+          <!-- 87 degrees across, which is what Intel publish for the D405. -->
+          <horizontal_fov>1.518</horizontal_fov>
+          <!-- One of the camera's own stream sizes, in its real 16:9 shape.
+               The shape has to be right, because Gazebo works the vertical
+               field of view out from it: at 4:3 this camera would appear to
+               see 71 degrees up and down instead of the 56 it really sees.
+               The size is the smallest real mode that still resolves the
+               table finely enough. A wide lens spreads its pixels over more
+               ground, so this camera needs more of them than the 60 degree
+               one it replaced: at 424 x 240 a pixel covers 2.0 mm of table
+               from the survey height, which is coarser than the millimetre
+               the measurements are reported to. At 640 x 360 it covers
+               1.33 mm, which is fine, and the frames are still small enough
+               to cross the ROS bridge comfortably. -->
           <image>
-            <width>320</width>
-            <height>240</height>
+            <width>640</width>
+            <height>360</height>
             <format>R8G8B8</format>
           </image>
+          <!-- The camera's real working range. Modelling it as a hard limit is
+               stricter than the hardware, which returns noisy depth outside it
+               rather than nothing, and that is deliberate: a limit the
+               simulator enforces is one that cannot be forgotten. It is also
+               what caps SURVEY_HEIGHT in arm/dimensions.py, because a survey
+               flown higher than this would be reading depth the camera cannot
+               stand behind. -->
           <clip>
-            <near>0.05</near>
-            <far>3.0</far>
+            <near>0.07</near>
+            <far>0.50</far>
           </clip>
-          <optical_frame_id>${prefix}wrist_camera_optical_frame</optical_frame_id>
+          <optical_frame_id>${prefix}wrist_camera_depth_optical_frame</optical_frame_id>
         </camera>
       </sensor>
